File: my devboard.kicad_pcb (KiCad board)
At the start: 2 copper layers, 21 x 51 mm, 33 parts, among them J1 USB_C_Receptacle_USB2.0_14P, J2 Conn_01x20, J3 Conn_01x20, J4 Conn_01x03, SW1 SW_Push, U1 RP2040, U2 MCP1700x-330xxTT, U3 W25Q16JVZPIQ, Y1 12 MHz

Commit message: done
Parts:
- added ?: LOGO, Rocket_solder:hackclub, B.Cu at (120.6, 100.8)
- added ?: LOGO, Rocket_solder:orph, B.Cu at (120.0, 75.1)
- added ?: LOGO, Rocket_solder4:qr_insta, B.Cu at (115.0, 70.0)
- added G***: LOGO, Rocket_solder:hmm, F.Cu at (120.0, 99.0)
- added G***: LOGO, Rocket_solder:purrrr, B.Cu at (120.0, 60.0)
- added G***: LOGO, Rocket_solder:linux, B.Cu at (119.1, 91.3)
- moved C16 0.78 mm to (122.8, 94.0)
- moved C12 0.30 mm to (122.9, 90.7)
Routing:
- net GND: track 41.7 -> 165.7 mm, vias 12 -> 26
- net GPIO15: track 25.5 -> 22.4 mm
- net XIN: track 19.4 -> 20.7 mm, vias 0 -> 1
- net SWCLK: track 21.6 -> 20.4 mm
- net GPIO04: track 19.9 -> 18.8 mm
- net QSPI_SS: track 12.5 -> 13.1 mm
Other:
- board text added: "Nitish"
